File: 01_spi_pont_H.sch (KiCad schematic (older format))
At the start: 9 parts, among them J1 Conn_01x10, J2 Conn_01x10, U1 NCV7708BDWR2G

Commit message: maj librairie
Parts:
- U1: symbol chimere_symbol:NCV7708BDWR2G -> Chimere_comps:NCV7708BDWR2G
Changed lines of the file:
@@
 $EndDescr
 $Comp
-L chimere_symbol:NCV7708BDWR2G U1
+L Chimere_comps:NCV7708BDWR2G U1
 U 1 1 5E98C0BB
 P 4100 2800
